Commit message: changes

File: description/urdf/moving_box_description.urdf (robot description, URDF)
Before this commit: robot None, 8 links, 7 joints
Joints:
- added joint gps_joint: type fixed, parent base_link, child gps_link, origin xyz=0 0 0 rpy=0 0 0

Commit message: changes

File: description/urdf/moving_box_description.urdf (robot description, URDF)
Before this commit: robot None, 8 links, 8 joints
Joints:
- removed joint gps_joint
