Commit message: gazebo

File: description/urdf/gazebo_control.xacro (robot description, xacro)
@@ -4,5 +4,18 @@
     <gazebo>
         <plugin name="diff_drive" filename="libgazebo_ros_diff_drive.so">
-            moving_box_hardware/MovingBoxHardware
+            <!-- Wheel Information -->
+            <left_joint>left_wheel_joint</left_joint>
+            <right_joint>right_wheel_joint</right_joint>
+            <wheel_separation>0.297</wheel_separation>
+            <wheel_diameter>0.066</wheel_diameter>
+            <!-- Limits -->
+            <max_wheel_torque>200</max_wheel_torque>
+            <max_wheel_acceleration>10.0</max_wheel_acceleration>
+            <!-- Output -->
+            <odometry_frame>odom</odometry_frame>
+            <robot_base_frame>base_link</robot_base_frame>
+            <publish_odom>true</publish_odom>
+            <publish_odom_tf>true</publish_odom_tf>
+            <publish_wheel_tf>true</publish_wheel_tf>
         </plugin>
     </gazebo>

File: description/urdf/lidar.xacro (robot description, xacro)
@@ -4,5 +4,5 @@
         <parent link="chassis"/>
         <child link="laser_frame"/>
-        <origin xyz="0.65 0 0.05" rpy="0 0 0"/>
+        <origin xyz="0.65 0 0.05" rpy="0 0 ${pi}"/>
     </joint>
     <link name="laser_frame">

File: description/urdf/moving_box.urdf.xacro (robot description, xacro)
@@ -4,8 +4,13 @@
   <xacro:arg name="prefix" default="" />
   <xacro:arg name="sim_mode" default="false"/>
+  <xacro:arg name="use_ros2_control" default="true"/>
   <xacro:include filename="$(find moving_box_hardware)/urdf/moving_box_description.urdf" />
   <!-- Import diffbot ros2_control description -->
-  <xacro:include filename="$(find moving_box_hardware)/ros2_control/moving_box.ros2_control.xacro" />
-  <!-- <xacro:include filename="gazebo_control.xacro"/> -->
+  <xacro:if value="$(arg use_ros2_control)">
+      <xacro:include filename="$(find moving_box_hardware)/ros2_control/moving_box.ros2_control.xacro" />
+  </xacro:if>
+  <xacro:unless value="$(arg use_ros2_control)">
+      <xacro:include filename="gazebo_control.xacro"/>
+  </xacro:unless>
   <xacro:include filename="lidar.xacro" />
   <!-- <xacro:include filename="sensors.xacro" /> -->
