Commit message: latency

File: description/urdf/lidar.xacro (robot description, xacro)
@@ -2,12 +2,12 @@
 <robot xmlns:xacro="http://www.ros.org/wiki/xacro" >
     <joint name="laser_joint" type="fixed">
-        <parent link="chassis"/>
+        <parent link="base_link"/>
         <child link="laser_frame"/>
-        <origin xyz="0.65 0 0.05" rpy="0 0 ${pi}"/>
+        <origin xyz="0 0 0.26" rpy="0 0 ${pi}"/>
     </joint>
     <link name="laser_frame">
         <visual>
             <geometry>
-                <cylinder radius="0.05" length="0.04"/>
+                <cylinder radius="0.03" length="0.03"/>
             </geometry>
             <material name="red"/>
@@ -15,8 +15,8 @@
         <collision>
             <geometry>
-                <cylinder radius="0.05" length="0.04"/>
+                <cylinder radius="0.03" length="0.03"/>
             </geometry>
         </collision>
-        <xacro:inertial_cylinder mass="2.0" length="0.04" radius="0.05">
+        <xacro:inertial_cylinder mass="1.0" length="0.03" radius="0.03">
             <origin xyz="0 0 0" rpy="0 0 0"/>
         </xacro:inertial_cylinder>

File: description/urdf/moving_box_description.urdf (robot description, URDF)
Before this commit: robot None, 8 links, 7 joints
Links:
- added link lidar_stick; collision box size=${lidar_stick_length} ${lidar_stick_width} ${lidar_stick_he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; visual box size=${lidar_stick_length} ${lidar_stick_width} ${lidar_stick_he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
Joints:
- added joint lidar_stick_joint: type fixed, parent base_link, child lidar_stick, origin xyz=0 0 0.125
